Commit message: debug-rrt

File: source/weldRobot/weldRobot/assets/robot-model/ur5e_with_pen.urdf (robot description, URDF)
Before this commit: robot ur5e_pen, 12 links, 11 joints
Joints:
- joint pen_link-tool0_fixed_joint: origin xyz=0 0 0.14 rpy=0 0 0 -> xyz=0 0 0.145 rpy=0 0 0

Commit message: sim stl

File: source/weldRobot/weldRobot/assets/robot-model/ur5e_with_pen.urdf (robot description, URDF)
Before this commit: robot ur5e_pen, 12 links, 11 joints
Joints:
- joint pen_link-tool0_fixed_joint: origin xyz=0 0 0.145 rpy=0 0 0 -> xyz=0 0 0.14 rpy=0 0 0
